Commit message: Xacro

File: src/urdf_test/urdf/my_robot.xacro (robot description, xacro)
@@ -1,4 +1,5 @@
 <?xml version="1.0"?>
-<robot name="my_robot">
+<robot name="my_robot" xmlns:xacro="http://www.ros.org/wiki/xacro" >
+    <xacro:property name="base_length" value="0.6" />
     <material name="blue">
         <color rgba="0 0 0.6 1" />
@@ -8,7 +9,7 @@
         <visual>
             <geometry>
-                <box size="0.6 0.4 0.2"/>
-            </geometry>1
-            <origin xyz="0 0 0.1" rpy="0 0 0"/>
+                <box size="${base_length} ${base_length / 1.5} ${base_length / 3.0}"/>
+            </geometry>
+            <origin xyz="0 0 ${base_length / 6.0}" rpy="0 0 0"/>
             <material name="blue" />
         </visual>
@@ -17,7 +18,7 @@
         <visual>
             <geometry>
-                <cylinder radius="0.1" length="0.07"/>
+                <cylinder radius="${base_length / 6.0}" length="${base_length / 12.0}"/>
             </geometry>
-            <origin xyz="0 0 0" rpy="1.57 0 0" />
+            <origin xyz="0 0 0" rpy="${pi / 2.0} 0 0" />
         </visual>
     </link>
@@ -25,7 +26,7 @@
         <visual>
             <geometry>
-                <cylinder radius="0.1" length="0.07" />
+                <cylinder radius="${base_length / 6.0}" length="${base_length / 12.0}" />
             </geometry>
-            <origin xyz="0 0 0" rpy="1.57 0 0" />
+            <origin xyz="0 0 0" rpy="${pi / 2.0} 0 0" />
         </visual>
     </link>
@@ -33,5 +34,5 @@
         <visual>
             <geometry>
-                <sphere radius="0.05" />
+                <sphere radius="${base_length / 12.0}" />
             </geometry>
             <origin xyz="0 0 0" rpy="0 0 0" />
@@ -41,5 +42,5 @@
         <parent link="base_link" />
         <child link="right_wheel_link" />
-        <origin xyz="-0.15 0.235 0" rpy="0 0 0" />
+        <origin xyz="${-base_length / 4.0} ${base_length / 2.55} 0" rpy="0 0 0" />
         <axis xyz="0 1 0" />
     </joint>
@@ -47,5 +48,5 @@
         <parent link="base_link" />
         <child link="left_wheel_link" />
-        <origin xyz="-0.15 -0.235 0" rpy="0 0 0" />
+        <origin xyz="${-base_length / 4.0} ${-base_length / 2.55} 0" rpy="0 0 0" />
         <axis xyz="0 1 0" />
     </joint>
@@ -53,5 +54,5 @@
         <parent link="base_link" />
         <child link="castor_wheel_link" />
-        <origin xyz="0.22 0 -0.045" rpy="0 0 0" />
+        <origin xyz="${base_length / 3.0} 0 ${-base_length / 13.3}" rpy="0 0 0" />
     </joint>
     <joint name="base_joint" type="fixed">
