Commit message: Gazebo

File: install/urdf_test/share/urdf_test/urdf/joints.xacro (robot description, xacro)
@@ -10,9 +10,19 @@
                 <origin xyz="0 0 0" rpy="${pi / 2.0} 0 0" />
             </visual>
+            <collision>
+                <geometry>
+                    <cylinder radius="${base_length / 6.0}" length="${base_length / 12.0}"/>
+                </geometry>
+                <origin xyz="0 0 0" rpy="${pi / 2.0} 0 0" />
+            </collision>
+            <inertial>
+                <mass value="0.5"/>
+                <inertia ixx="0.001" iyy="0.001" izz="0.001" ixy="0.0" ixz="0.0" iyz="0.0"/>
+            </inertial>
         </link>
     </xacro:macro>
     <xacro:wheel_link name="left"/>
     <xacro:wheel_link name="right"/>
-    <link name="base_footprint" />
+    <link name="base_footprint"/>
     <link name="base_link">
         <visual>
@@ -23,4 +33,14 @@
             <material name="blue" />
         </visual>
+        <collision>
+            <geometry>
+                <box size="${base_length} ${base_length / 1.5} ${base_length / 3.0}"/>
+            </geometry>
+            <origin xyz="0 0 ${base_length / 6.0}" rpy="0 0 0"/>
+        </collision>
+        <inertial>
+            <mass value="5.0"/>
+            <inertia ixx="0.1" iyy="0.1" izz="0.1" ixy="0.0" ixz="0.0" iyz="0.0"/>
+        </inertial>
     </link>
     <link name="castor_wheel_link">
@@ -31,4 +51,14 @@
             <origin xyz="0 0 0" rpy="0 0 0" />
         </visual>
+        <collision>
+            <geometry>
+                <sphere radius="${base_length / 12.0}" />
+            </geometry>
+            <origin xyz="0 0 0" rpy="0 0 0" />
+        </collision>
+        <inertial>
+            <mass value="0.2"/>
+            <inertia ixx="0.0001" iyy="0.0001" izz="0.0001" ixy="0.0" ixz="0.0" iyz="0.0"/>
+        </inertial>
     </link>
 </robot>

File: install/urdf_test/share/urdf_test/urdf/my_robot.xacro (robot description, xacro)
@@ -10,5 +10,5 @@
             <origin xyz="0.0 0.0 0.0" rpy="0.0 0.0 0.0" />
             <geometry>
-                <mesh filename="package://urdf_test/meshes/base.stl" scale="0.001 0.001 0.001" />
+                <mesh filename="model://urdf_test/meshes/base.stl" scale="0.001 0.001 0.001" />
             </geometry>
         </visual>
@@ -16,5 +16,5 @@
             <origin xyz="0.0 0.0 0.0" rpy="0.0 0.0 0.0" />
             <geometry>
-                <mesh filename="package://urdf_test/meshes/base.stl" scale="0.001 0.001 0.001" />
+                <mesh filename="model://urdf_test/meshes/base.stl" scale="0.001 0.001 0.001" />
             </geometry>
         </collision>
@@ -29,5 +29,5 @@
             <origin xyz="0.05050000000000001 -1.6653345369377347e-18 0.005" rpy="3.141592653589793 -0.0 0.0" />
             <geometry>
-                <mesh filename="package://urdf_test/meshes/steering.stl" scale="0.001 0.001 0.001" />
+                <mesh filename="model://urdf_test/meshes/steering.stl" scale="0.001 0.001 0.001" />
             </geometry>
         </visual>
@@ -35,5 +35,5 @@
             <origin xyz="0.05050000000000001 -1.6653345369377347e-18 0.005" rpy="3.141592653589793 -0.0 0.0" />
             <geometry>
-                <mesh filename="package://urdf_test/meshes/steering.stl" scale="0.001 0.001 0.001" />
+                <mesh filename="model://urdf_test/meshes/steering.stl" scale="0.001 0.001 0.001" />
             </geometry>
         </collision>
@@ -48,5 +48,5 @@
             <origin xyz="-0.06302599985826682 -0.003489789468550507 0.0029999999999999983" rpy="-1.5707963267948966 -0.0 3.141592653589793" />
             <geometry>
-                <mesh filename="package://urdf_test/meshes/front_wheel.stl" scale="0.001 0.001 0.001" />
+                <mesh filename="model://urdf_test/meshes/front_wheel.stl" scale="0.001 0.001 0.001" />
             </geometry>
         </visual>
@@ -54,5 +54,5 @@
             <origin xyz="-0.06302599985826682 -0.003489789468550507 0.0029999999999999983" rpy="-1.5707963267948966 -0.0 3.141592653589793" />
             <geometry>
-                <mesh filename="package://urdf_test/meshes/front_wheel.stl" scale="0.001 0.001 0.001" />
+                <mesh filename="model://urdf_test/meshes/front_wheel.stl" scale="0.001 0.001 0.001" />
             </geometry>
         </collision>
@@ -67,5 +67,5 @@
             <origin xyz="0.026000000372529027 -3.1840817234047667e-18 -0.02" rpy="1.5707963267948966 -0.0 3.141592653589793" />
             <geometry>
-                <mesh filename="package://urdf_test/meshes/right_wheel.stl" scale="0.001 0.001 0.001" />
+                <mesh filename="model://urdf_test/meshes/right_wheel.stl" scale="0.001 0.001 0.001" />
             </geometry>
         </visual>
@@ -73,5 +73,5 @@
             <origin xyz="0.026000000372529027 -3.1840817234047667e-18 -0.02" rpy="1.5707963267948966 -0.0 3.141592653589793" />
             <geometry>
-                <mesh filename="package://urdf_test/meshes/right_wheel.stl" scale="0.001 0.001 0.001" />
+                <mesh filename="model://urdf_test/meshes/right_wheel.stl" scale="0.001 0.001 0.001" />
             </geometry>
         </collision>
@@ -86,5 +86,5 @@
             <origin xyz="-0.004341204506362234 0.02462019419217468 -0.02" rpy="-1.5707963267948966 -0.0 -1.396263401595464" />
             <geometry>
-                <mesh filename="package://urdf_test/meshes/left_wheel.stl" scale="0.001 0.001 0.001" />
+                <mesh filename="model://urdf_test/meshes/left_wheel.stl" scale="0.001 0.001 0.001" />
             </geometry>
         </visual>
@@ -92,5 +92,5 @@
             <origin xyz="-0.004341204506362234 0.02462019419217468 -0.02" rpy="-1.5707963267948966 -0.0 -1.396263401595464" />
             <geometry>
-                <mesh filename="package://urdf_test/meshes/left_wheel.stl" scale="0.001 0.001 0.001" />
+                <mesh filename="model://urdf_test/meshes/left_wheel.stl" scale="0.001 0.001 0.001" />
             </geometry>
         </collision>
@@ -105,5 +105,5 @@
             <origin xyz="-1.1102230246251566e-18 0.0 -0.023" rpy="0.0 -0.0 0.0" />
             <geometry>
-                <mesh filename="package://urdf_test/meshes/arm_1.stl" scale="0.001 0.001 0.001" />
+                <mesh filename="model://urdf_test/meshes/arm_1.stl" scale="0.001 0.001 0.001" />
             </geometry>
         </visual>
@@ -111,5 +111,5 @@
             <origin xyz="-1.1102230246251566e-18 0.0 -0.023" rpy="0.0 -0.0 0.0" />
             <geometry>
-                <mesh filename="package://urdf_test/meshes/arm_1.stl" scale="0.001 0.001 0.001" />
+                <mesh filename="model://urdf_test/meshes/arm_1.stl" scale="0.001 0.001 0.001" />
             </geometry>
         </collision>
@@ -124,5 +124,5 @@
             <origin xyz="-0.05149999658483846 3.7085770201170125e-18 0.004980669999999999" rpy="3.141592653589793 -1.5707963267948966 0" />
             <geometry>
-                <mesh filename="package://urdf_test/meshes/arm_2.stl" scale="0.001 0.001 0.001" />
+                <mesh filename="model://urdf_test/meshes/arm_2.stl" scale="0.001 0.001 0.001" />
             </geometry>
         </visual>
@@ -130,5 +130,5 @@
             <origin xyz="-0.05149999658483846 3.7085770201170125e-18 0.004980669999999999" rpy="3.141592653589793 -1.5707963267948966 0" />
             <geometry>
-                <mesh filename="package://urdf_test/meshes/arm_2.stl" scale="0.001 0.001 0.001" />
+                <mesh filename="model://urdf_test/meshes/arm_2.stl" scale="0.001 0.001 0.001" />
             </geometry>
         </collision>
@@ -143,5 +143,5 @@
             <origin xyz="-0.09049999658483845 2.259060191846725e-18 0.003979455781202988" rpy="1.232595164407831e-32 1.5707963267948966 0" />
             <geometry>
-                <mesh filename="package://urdf_test/meshes/arm_3.stl" scale="0.001 0.001 0.001" />
+                <mesh filename="model://urdf_test/meshes/arm_3.stl" scale="0.001 0.001 0.001" />
             </geometry>
         </visual>
@@ -149,5 +149,5 @@
             <origin xyz="-0.09049999658483845 2.259060191846725e-18 0.003979455781202988" rpy="1.232595164407831e-32 1.5707963267948966 0" />
             <geometry>
-                <mesh filename="package://urdf_test/meshes/arm_3.stl" scale="0.001 0.001 0.001" />
+                <mesh filename="model://urdf_test/meshes/arm_3.stl" scale="0.001 0.001 0.001" />
             </geometry>
         </collision>
@@ -162,5 +162,5 @@
             <origin xyz="0.0543908059196748 -0.12899144399999998 -0.003311543941894128" rpy="-1.5707963267948963 -0.0 0.0" />
             <geometry>
-                <mesh filename="package://urdf_test/meshes/gripper_gear_1.stl" scale="0.001 0.001 0.001" />
+                <mesh filename="model://urdf_test/meshes/gripper_gear_1.stl" scale="0.001 0.001 0.001" />
             </geometry>
         </visual>
@@ -168,5 +168,5 @@
             <origin xyz="0.0543908059196748 -0.12899144399999998 -0.003311543941894128" rpy="-1.5707963267948963 -0.0 0.0" />
             <geometry>
-                <mesh filename="package://urdf_test/meshes/gripper_gear_1.stl" scale="0.001 0.001 0.001" />
+                <mesh filename="model://urdf_test/meshes/gripper_gear_1.stl" scale="0.001 0.001 0.001" />
             </geometry>
         </collision>
@@ -181,5 +181,5 @@
             <origin xyz="0.06143864417246264 -0.12899634400000004 -0.00331643944132532" rpy="-1.5707963267948963 -0.0 0.0" />
             <geometry>
-                <mesh filename="package://urdf_test/meshes/gripper_gear_2.stl" scale="0.001 0.001 0.001" />
+                <mesh filename="model://urdf_test/meshes/gripper_gear_2.stl" scale="0.001 0.001 0.001" />
             </geometry>
         </visual>
@@ -187,5 +187,5 @@
             <origin xyz="0.06143864417246264 -0.12899634400000004 -0.00331643944132532" rpy="-1.5707963267948963 -0.0 0.0" />
             <geometry>
-                <mesh filename="package://urdf_test/meshes/gripper_gear_2.stl" scale="0.001 0.001 0.001" />
+                <mesh filename="model://urdf_test/meshes/gripper_gear_2.stl" scale="0.001 0.001 0.001" />
             </geometry>
         </collision>
