Commit message: Gazebo

File: install/urdf_test/share/urdf_test/urdf/example.xacro (robot description, xacro)
@@ -5,4 +5,24 @@
     <xacro:include filename="links.xacro" />
     <xacro:property name="base_length" value="0.6" />
+    <gazebo reference="castor_wheel_link">
+        <mu1>0.1</mu1>
+        <mu2>0.1</mu2>
+    </gazebo>
+    <gazebo>
+        <plugin name="gz::sim::systems::DiffDrive" filename="gz-sim-diff-drive-system">
+            <left_joint>base_left_wheel_joint</left_joint>
+            <right_joint>base_right_wheel_joint</right_joint>
+            <wheel_separation>0.34</wheel_separation>
+            <wheel_radius>0.1</wheel_radius>
+            <frame_id>odom</frame_id>
+            <child_frame_id>base_footprint</child_frame_id>
+        </plugin>
+    </gazebo>
+    <gazebo>
+        <plugin name = "gz::sim::systems::JointStatePublisher" filename="gz-sim-joint-state-publisher-system">
+            <joint_name>base_left_wheel_joint</joint_name>
+            <joint_name>base_right_wheel_joint</joint_name>
+        </plugin>
+    </gazebo>
     <!-- <xacro:macro name="example_macro" params="a b c">
         stuff

File: install/urdf_test/share/urdf_test/urdf/links.xacro (robot description, xacro)
@@ -2,13 +2,13 @@
 <robot xmlns:xacro="http://www.ros.org/wiki/xacro" >
     <xacro:property name="base_length" value="0.6" />
+    <joint name="base_left_wheel_joint" type="continuous">
+        <parent link="base_link" />
+        <child link="left_wheel_link" />
+        <origin xyz="${-base_length / 4.0} ${base_length / 2.55} 0" rpy="0 0 0" />
+        <axis xyz="0 1 0" />
+    </joint>
     <joint name="base_right_wheel_joint" type="continuous">
         <parent link="base_link" />
         <child link="right_wheel_link" />
-        <origin xyz="${-base_length / 4.0} ${base_length / 2.55} 0" rpy="0 0 0" />
-        <axis xyz="0 1 0" />
-    </joint>
-    <joint name="base_left_wheel_link" type="continuous">
-        <parent link="base_link" />
-        <child link="left_wheel_link" />
         <origin xyz="${-base_length / 4.0} ${-base_length / 2.55} 0" rpy="0 0 0" />
         <axis xyz="0 1 0" />

File: src/urdf_test/urdf/example.xacro (robot description, xacro)
@@ -11,14 +11,8 @@
     <gazebo>
         <plugin name="gz::sim::systems::DiffDrive" filename="gz-sim-diff-drive-system">
-            <left_joint>left_wheel_joint</left_joint>
-            <right_joint>right_wheel_joint</right_joint>
+            <left_joint>base_left_wheel_joint</left_joint>
+            <right_joint>base_right_wheel_joint</right_joint>
             <wheel_separation>0.34</wheel_separation>
             <wheel_radius>0.1</wheel_radius>
-            <topic>/cmd_vel</topic>
-            <odometry_topic>/odom</odometry_topic>
-            <odometry_frame>odom</odometry_frame>
-            <robot_base_frame>base_link</robot_base_frame>
-            <update_rate>100.0</update_rate>
-            <gaussian_noise>0.0</gaussian_noise>
             <frame_id>odom</frame_id>
             <child_frame_id>base_footprint</child_frame_id>

Commit message: Gazebo Sensors

File: install/urdf_test/share/urdf_test/urdf/example.xacro (robot description, xacro)
@@ -4,4 +4,5 @@
     <xacro:include filename="joints.xacro" />
     <xacro:include filename="links.xacro" />
+    <xacro:include filename="sensors.xacro" />
     <xacro:property name="base_length" value="0.6" />
     <gazebo reference="castor_wheel_link">

File: install/urdf_test/share/urdf_test/urdf/materials.xacro (robot description, xacro)
@@ -4,3 +4,6 @@
         <color rgba="0 0 0.6 1" />
     </material>
+    <material name="red">
+        <color rgba="0.6 0 0 1" />
+    </material>
 </robot>
