Commit message: Xacro Updates

File: install/urdf_test/share/urdf_test/urdf/my_robot.xacro (robot description, xacro)
@@ -1,64 +1,13 @@
 <?xml version="1.0"?>
 <robot name="my_robot" xmlns:xacro="http://www.ros.org/wiki/xacro" >
+    <xacro:include filename="materials.xacro" />
+    <xacro:include filename="links.xacro" />
+    <xacro:include filename="joints.xacro" />
     <xacro:property name="base_length" value="0.6" />
-    <material name="blue">
-        <color rgba="0 0 0.6 1" />
-    </material>
-    <link name="base_footprint" />
-    <link name="base_link">
-        <visual>
-            <geometry>
-                <box size="${base_length} ${base_length / 1.5} ${base_length / 3.0}"/>
-            </geometry>
-            <origin xyz="0 0 ${base_length / 6.0}" rpy="0 0 0"/>
-            <material name="blue" />
-        </visual>
-    </link>
-    <link name="right_wheel_link">
-        <visual>
-            <geometry>
-                <cylinder radius="${base_length / 6.0}" length="${base_length / 12.0}"/>
-            </geometry>
-            <origin xyz="0 0 0" rpy="${pi / 2.0} 0 0" />
-        </visual>
-    </link>
-    <link name="left_wheel_link">
-        <visual>
-            <geometry>
-                <cylinder radius="${base_length / 6.0}" length="${base_length / 12.0}" />
-            </geometry>
-            <origin xyz="0 0 0" rpy="${pi / 2.0} 0 0" />
-        </visual>
-    </link>
-    <link name="castor_wheel_link">
-        <visual>
-            <geometry>
-                <sphere radius="${base_length / 12.0}" />
-            </geometry>
-            <origin xyz="0 0 0" rpy="0 0 0" />
-        </visual>
-    </link>
-    <joint name="base_right_wheel_joint" type="continuous">
-        <parent link="base_link" />
-        <child link="right_wheel_link" />
-        <origin xyz="${-base_length / 4.0} ${base_length / 2.55} 0" rpy="0 0 0" />
-        <axis xyz="0 1 0" />
-    </joint>
-    <joint name="base_left_wheel_link" type="continuous">
-        <parent link="base_link" />
-        <child link="left_wheel_link" />
-        <origin xyz="${-base_length / 4.0} ${-base_length / 2.55} 0" rpy="0 0 0" />
-        <axis xyz="0 1 0" />
-    </joint>
-    <joint name="base_castor_wheel_link" type="fixed">
-        <parent link="base_link" />
-        <child link="castor_wheel_link" />
-        <origin xyz="${base_length / 3.0} 0 ${-base_length / 13.3}" rpy="0 0 0" />
-    </joint>
-    <joint name="base_joint" type="fixed">
-        <parent link="base_footprint" />
-        <child link="base_link" />
-        <origin xyz="0 0 0.1" rpy="0 0 0" />
-    </joint>
+    <!-- <xacro:macro name="example_macro" params="a b c">
+        stuff
+        using ${a} etc...
+    </xacro:macro> -->
+    <!-- <xacro:example_macro a="2" b="3" c="1" -->
     <!-- <joint name="base_second_joint" type="continuous">
         <parent link="base_link" />

Commit message: Test URDF export from Fusion 360.

File: install/urdf_test/share/urdf_test/urdf/my_robot.xacro (robot description, xacro)
@@ -1,25 +1,123 @@
-<?xml version="1.0"?>
-<robot name="my_robot" xmlns:xacro="http://www.ros.org/wiki/xacro" >
-    <xacro:include filename="materials.xacro" />
-    <xacro:include filename="links.xacro" />
-    <xacro:include filename="joints.xacro" />
-    <xacro:property name="base_length" value="0.6" />
-    <!-- <xacro:macro name="example_macro" params="a b c">
-        stuff
-        using ${a} etc...
-    </xacro:macro> -->
-    <!-- <xacro:example_macro a="2" b="3" c="1" -->
-    <!-- <joint name="base_second_joint" type="continuous">
-        <parent link="base_link" />
-        <child link="second_link" />
-        <origin xyz="0 0 0.2" rpy="0 0 0" />
-        <axis xyz="0 0 1" />
-    </joint> -->
-    <!-- <joint name="base_second_joint" type="prismatic">
-        <parent link="base_link" />
-        <child link="second_link" />
-        <origin xyz="0 0 0.2" rpy="0 0 0" />
-        <axis xyz="1 0 0" />
-        <limit lower="0.0" upper="0.5" velocity="100" effort="100" />
-    </joint> -->
+<?xml version='1.0' encoding='utf-8'?>
+<robot name="(Unsaved)">
+    <link name="base">
+        <inertial>
+            <origin xyz="0.0008223144260215306 1.973712041524325e-10 0.009266969689636867" rpy="0.0 0.0 0.0" />
+            <mass value="0.4573772989307287" />
+            <inertia ixx="6.683277879258534e-05" iyy="0.00025359566623103314" izz="0.00029307903194205145" ixy="3.21815854370631e-12" iyz="4.1009766970174006e-14" ixz="-7.073165358312158e-08" />
+        </inertial>
+        <visual name="base_visual">
+            <origin xyz="0.0 0.0 0.0" rpy="0.0 0.0 0.0" />
+            <geometry>
+                <mesh filename="package://urdf_test/meshes/base.stl" scale="0.001 0.001 0.001" />
+            </geometry>
+        </visual>
+        <collision name="base_collision">
+            <origin xyz="0.0 0.0 0.0" rpy="0.0 0.0 0.0" />
+            <geometry>
+                <mesh filename="package://urdf_test/meshes/base.stl" scale="0.001 0.001 0.001" />
+            </geometry>
+        </collision>
+    </link>
+    <link name="steering">
+        <inertial>
+            <origin xyz="-0.0037663810496018704 2.6816932522572467e-10 0.004608964195140794" rpy="0.0 -0.0 0.0" />
+            <mass value="0.0022331707953948026" />
+            <inertia ixx="3.5663821715718204e-08" iyy="5.943179529055522e-08" izz="5.871726437717775e-08" ixy="6.841246453702055e-15" iyz="-1.1530872167369278e-15" ixz="1.921765263778425e-08" />
+        </inertial>
+        <visual name="steering_visual">
+            <origin xyz="0.05050000000000001 -1.6653345369377347e-18 0.005" rpy="3.141592653589793 -0.0 0.0" />
+            <geometry>
+                <mesh filename="package://urdf_test/meshes/steering.stl" scale="0.001 0.001 0.001" />
+            </geometry>
+        </visual>
+        <collision name="steering_collision">
+            <origin xyz="0.05050000000000001 -1.6653345369377347e-18 0.005" rpy="3.141592653589793 -0.0 0.0" />
+            <geometry>
+                <mesh filename="package://urdf_test/meshes/steering.stl" scale="0.001 0.001 0.001" />
+            </geometry>
+        </collision>
+    </link>
+    <link name="front_wheel">
+        <inertial>
+            <origin xyz="8.866190892575787e-10 7.450580596923828e-11 0.003000000000000002" rpy="0.0 -0.0 0.0" />
+            <mass value="0.008303387259265533" />
+            <inertia ixx="1.4047457758420725e-07" iyy="1.4047457758420304e-07" izz="2.3559678534938288e-07" ixy="-4.235164736271502e-22" iyz="-1.7697461564018615e-23" ixz="-3.7843359830029504e-22" />
+        </inertial>
+        <visual name="front_wheel_visual">
+            <origin xyz="-0.06302599985826682 -0.003489789468550507 0.0029999999999999983" rpy="-1.5707963267948966 -0.0 3.141592653589793" />
+            <geometry>
+                <mesh filename="package://urdf_test/meshes/front_wheel.stl" scale="0.001 0.001 0.001" />
+            </geometry>
+        </visual>
+        <collision name="front_wheel_collision">
+            <origin xyz="-0.06302599985826682 -0.003489789468550507 0.0029999999999999983" rpy="-1.5707963267948966 -0.0 3.141592653589793" />
+            <geometry>
+                <mesh filename="package://urdf_test/meshes/front_wheel.stl" scale="0.001 0.001 0.001" />
+            </geometry>
+        </collision>
+    </link>
+    <link name="right_wheel">
+        <inertial>
+            <origin xyz="0.0 -4.930380657631324e-34 0.0029999999999999983" rpy="0.0 -0.0 0.0" />
+            <mass value="0.017542070720840106" />
+            <inertia ixx="5.717776098641495e-07" iyy="5.717776098641716e-07" izz="1.0425458548287574e-06" ixy="2.4003235141830388e-36" iyz="-3.486100297322995e-22" ixz="8.470329472543003e-22" />
+        </inertial>
+        <visual name="right_wheel_visual">
+            <origin xyz="0.026000000372529027 -3.1840817234047667e-18 -0.02" rpy="1.5707963267948966 -0.0 3.141592653589793" />
+            <geometry>
+                <mesh filename="package://urdf_test/meshes/right_wheel.stl" scale="0.001 0.001 0.001" />
+            </geometry>
+        </visual>
+        <collision name="right_wheel_collision">
+            <origin xyz="0.026000000372529027 -3.1840817234047667e-18 -0.02" rpy="1.5707963267948966 -0.0 3.141592653589793" />
+            <geometry>
+                <mesh filename="package://urdf_test/meshes/right_wheel.stl" scale="0.001 0.001 0.001" />
+            </geometry>
+        </collision>
+    </link>
+    <link name="left_wheel">
+        <inertial>
+            <origin xyz="0.0 4.440892098500626e-18 0.0030000000000000027" rpy="0.0 -0.0 0.0" />
+            <mass value="0.017542070720840106" />
+            <inertia ixx="5.717776098641648e-07" iyy="5.717776098641461e-07" izz="1.0425458548287587e-06" ixy="4.2729574083186744e-21" iyz="4.039774140954686e-22" ixz="8.470329472543003e-22" />
+        </inertial>
+        <visual name="left_wheel_visual">
+            <origin xyz="-0.0043412045063622355 0.02462019419217468 -0.02" rpy="-1.5707963267948966 -0.0 -1.396263401595464" />
+            <geometry>
+                <mesh filename="package://urdf_test/meshes/left_wheel.stl" scale="0.001 0.001 0.001" />
+            </geometry>
+        </visual>
+        <collision name="left_wheel_collision">
+            <origin xyz="-0.0043412045063622355 0.02462019419217468 -0.02" rpy="-1.5707963267948966 -0.0 -1.396263401595464" />
+            <geometry>
+                <mesh filename="package://urdf_test/meshes/left_wheel.stl" scale="0.001 0.001 0.001" />
+            </geometry>
+        </collision>
+    </link>
+    <joint name="base_Revolute-1" type="revolute">
+        <origin xyz="-0.051 0.0 0.005" rpy="3.141592653589793 -0.0 0.0" />
+        <parent link="base" />
+        <child link="steering" />
+        <axis xyz="0.0 0.0 1.0" />
+        <limit lower="-1.570796" upper="1.570796" effort="1000000" velocity="1000000" />
+    </joint>
+    <joint name="base_Revolute-3" type="continuous">
+        <origin xyz="0.0075 -0.02 0.0" rpy="-1.5707963267948966 -0.0 3.141592653589793" />
+        <parent link="base" />
+        <child link="left_wheel" />
+        <axis xyz="0.0 0.0 1.0" />
+    </joint>
+    <joint name="base_Revolute-4" type="continuous">
+        <origin xyz="0.0075 0.02 0.0" rpy="-1.5707963267948966 -0.0 0.0" />
+        <parent link="base" />
+        <child link="right_wheel" />
+        <axis xyz="0.0 0.0 1.0" />
+    </joint>
+    <joint name="steering_Revolute-6" type="continuous">
+        <origin xyz="-0.012000000000000002 -0.003 0.01" rpy="1.5707963267948966 -0.0 3.141592653589793" />
+        <parent link="steering" />
+        <child link="front_wheel" />
+        <axis xyz="0.0 0.0 1.0" />
+    </joint>
 </robot>

Commit message: Robot Testing with URDF

File: install/urdf_test/share/urdf_test/urdf/my_robot.xacro (robot description, xacro)
@@ -1,9 +1,9 @@
 <?xml version='1.0' encoding='utf-8'?>
-<robot name="(Unsaved)">
+<robot name="ros2_robot_test1">
     <link name="base">
         <inertial>
-            <origin xyz="0.0008223144260215306 1.973712041524325e-10 0.009266969689636867" rpy="0.0 0.0 0.0" />
-            <mass value="0.4573772989307287" />
-            <inertia ixx="6.683277879258534e-05" iyy="0.00025359566623103314" izz="0.00029307903194205145" ixy="3.21815854370631e-12" iyz="4.1009766970174006e-14" ixz="-7.073165358312158e-08" />
+            <origin xyz="-0.00483946780539695 6.928044477352326e-10 0.009034319690654786" rpy="0.0 0.0 0.0" />
+            <mass value="0.1303009956887525" />
+            <inertia ixx="2.7313724606267886e-05" iyy="7.344400471054905e-05" izz="8.682097283779688e-05" ixy="2.7070518357774284e-12" iyz="2.0007738507830658e-14" ixz="-1.3092363029253664e-07" />
         </inertial>
         <visual name="base_visual">
@@ -22,7 +22,7 @@
     <link name="steering">
         <inertial>
-            <origin xyz="-0.0037663810496018704 2.6816932522572467e-10 0.004608964195140794" rpy="0.0 -0.0 0.0" />
+            <origin xyz="-0.0037663810496018613 2.6816932522572467e-10 0.004608964195140794" rpy="0.0 -0.0 0.0" />
             <mass value="0.0022331707953948026" />
-            <inertia ixx="3.5663821715718204e-08" iyy="5.943179529055522e-08" izz="5.871726437717775e-08" ixy="6.841246453702055e-15" iyz="-1.1530872167369278e-15" ixz="1.921765263778425e-08" />
+            <inertia ixx="3.5663821715718204e-08" iyy="5.943179529055607e-08" izz="5.871726437717775e-08" ixy="6.8412464972783024e-15" iyz="-1.1530872167369278e-15" ixz="1.9217652637784286e-08" />
         </inertial>
         <visual name="steering_visual">
@@ -62,5 +62,5 @@
             <origin xyz="0.0 -4.930380657631324e-34 0.0029999999999999983" rpy="0.0 -0.0 0.0" />
             <mass value="0.017542070720840106" />
-            <inertia ixx="5.717776098641495e-07" iyy="5.717776098641716e-07" izz="1.0425458548287574e-06" ixy="2.4003235141830388e-36" iyz="-3.486100297322995e-22" ixz="8.470329472543003e-22" />
+            <inertia ixx="5.717776098641495e-07" iyy="5.717776098641699e-07" izz="1.0425458548287574e-06" ixy="2.4435680572714544e-36" iyz="-3.486100297322995e-22" ixz="1.4823076576950256e-21" />
         </inertial>
         <visual name="right_wheel_visual">
@@ -79,10 +79,10 @@
     <link name="left_wheel">
         <inertial>
-            <origin xyz="0.0 4.440892098500626e-18 0.0030000000000000027" rpy="0.0 -0.0 0.0" />
+            <origin xyz="1.3877787807814458e-18 4.440892098500626e-18 0.0030000000000000027" rpy="0.0 -0.0 0.0" />
             <mass value="0.017542070720840106" />
-            <inertia ixx="5.717776098641648e-07" iyy="5.717776098641461e-07" izz="1.0425458548287587e-06" ixy="4.2729574083186744e-21" iyz="4.039774140954686e-22" ixz="8.470329472543003e-22" />
+            <inertia ixx="5.717776098641648e-07" iyy="5.717776098641461e-07" izz="1.0425458548287591e-06" ixy="3.968580234205542e-21" iyz="4.039774140954686e-22" ixz="4.235164736271502e-22" />
         </inertial>
         <visual name="left_wheel_visual">
-            <origin xyz="-0.0043412045063622355 0.02462019419217468 -0.02" rpy="-1.5707963267948966 -0.0 -1.396263401595464" />
+            <origin xyz="-0.004341204506362234 0.02462019419217468 -0.02" rpy="-1.5707963267948966 -0.0 -1.396263401595464" />
             <geometry>
                 <mesh filename="package://urdf_test/meshes/left_wheel.stl" scale="0.001 0.001 0.001" />
@@ -90,7 +90,64 @@
         </visual>
         <collision name="left_wheel_collision">
-            <origin xyz="-0.0043412045063622355 0.02462019419217468 -0.02" rpy="-1.5707963267948966 -0.0 -1.396263401595464" />
+            <origin xyz="-0.004341204506362234 0.02462019419217468 -0.02" rpy="-1.5707963267948966 -0.0 -1.396263401595464" />
             <geometry>
                 <mesh filename="package://urdf_test/meshes/left_wheel.stl" scale="0.001 0.001 0.001" />
+            </geometry>
+        </collision>
+    </link>
+    <link name="arm_1">
+        <inertial>
+            <origin xyz="5.514138850609185e-14 4.52260766016217e-09 0.011800028069449754" rpy="0.0 -0.0 0.0" />
+            <mass value="0.02298483953953437" />
+            <inertia ixx="1.302346278933298e-06" iyy="1.3607994319911767e-06" izz="5.447043264270214e-07" ixy="8.772572149000581e-22" iyz="-1.0942767915434933e-12" ixz="1.2999131864653754e-17" />
+        </inertial>
+        <visual name="arm_1_visual">
+            <origin xyz="-1.1102230246251566e-18 0.0 -0.023" rpy="0.0 -0.0 0.0" />
+            <geometry>
+                <mesh filename="package://urdf_test/meshes/arm_1.stl" scale="0.001 0.001 0.001" />
+            </geometry>
+        </visual>
+        <collision name="arm_1_collision">
+            <origin xyz="-1.1102230246251566e-18 0.0 -0.023" rpy="0.0 -0.0 0.0" />
+            <geometry>
+                <mesh filename="package://urdf_test/meshes/arm_1.stl" scale="0.001 0.001 0.001" />
+            </geometry>
+        </collision>
+    </link>
+    <link name="arm_2">
+        <inertial>
+            <origin xyz="0.015555480853677217 2.260878411753778e-10 0.0049806690937104405" rpy="0.0 -0.0 0.0" />
+            <mass value="0.02207119901091111" />
+            <inertia ixx="2.752592908035583e-07" iyy="2.6715896972011874e-06" izz="2.660450936707386e-06" ixy="-8.440142306641492e-14" iyz="1.3735171472488167e-14" ixz="3.383607601166485e-13" />
+        </inertial>
+        <visual name="arm_2_visual">
+            <origin xyz="-0.05149999658483846 3.7085770201170125e-18 0.004980669999999999" rpy="3.141592653589793 -1.5707963267948966 0" />
+            <geometry>
+                <mesh filename="package://urdf_test/meshes/arm_2.stl" scale="0.001 0.001 0.001" />
+            </geometry>
+        </visual>
+        <collision name="arm_2_collision">
+            <origin xyz="-0.05149999658483846 3.7085770201170125e-18 0.004980669999999999" rpy="3.141592653589793 -1.5707963267948966 0" />
+            <geometry>
+                <mesh filename="package://urdf_test/meshes/arm_2.stl" scale="0.001 0.001 0.001" />
+            </geometry>
+        </collision>
+    </link>
+    <link name="arm_3">
+        <inertial>
+            <origin xyz="0.017021830705348132 2.2590601918467236e-18 0.003979455780812923" rpy="0.0 -0.0 0.0" />
+            <mass value="0.015207027813440301" />
+            <inertia ixx="1.1895476288949197e-07" iyy="1.9861577194252387e-06" izz="1.9861577267136794e-06" ixy="1.7430501486614956e-21" iyz="9.183549615799121e-41" ixz="-4.684356896112298e-17" />
+        </inertial>
+        <visual name="arm_3_visual">
+            <origin xyz="-0.09049999658483847 2.259060191846725e-18 0.003979455781202988" rpy="1.232595164407831e-32 1.5707963267948966 0" />
+            <geometry>
+                <mesh filename="package://urdf_test/meshes/arm_3.stl" scale="0.001 0.001 0.001" />
+            </geometry>
+        </visual>
+        <collision name="arm_3_collision">
+            <origin xyz="-0.09049999658483847 2.259060191846725e-18 0.003979455781202988" rpy="1.232595164407831e-32 1.5707963267948966 0" />
+            <geometry>
+                <mesh filename="package://urdf_test/meshes/arm_3.stl" scale="0.001 0.001 0.001" />
             </geometry>
         </collision>
@@ -104,5 +161,5 @@
     </joint>
     <joint name="base_Revolute-3" type="continuous">
-        <origin xyz="0.0075 -0.02 0.0" rpy="-1.5707963267948966 -0.0 3.141592653589793" />
+        <origin xyz="0.0025 -0.02 0.0" rpy="-1.5707963267948966 -0.0 3.141592653589793" />
         <parent link="base" />
         <child link="left_wheel" />
@@ -110,5 +167,5 @@
     </joint>
     <joint name="base_Revolute-4" type="continuous">
-        <origin xyz="0.0075 0.02 0.0" rpy="-1.5707963267948966 -0.0 0.0" />
+        <origin xyz="0.0025 0.02 0.0" rpy="-1.5707963267948966 -0.0 0.0" />
         <parent link="base" />
         <child link="right_wheel" />
@@ -121,3 +178,23 @@
         <axis xyz="0.0 0.0 1.0" />
     </joint>
+    <joint name="arm_1_Revolute-9" type="revolute">
+        <origin xyz="-0.0049806699999999995 0.0 0.02594445" rpy="-3.141592653589793 -1.5707963267948966 0" />
+        <parent link="arm_1" />
+        <child link="arm_2" />
+        <axis xyz="0.0 0.0 1.0" />
+        <limit lower="-1.570796" upper="1.570796" effort="1000000" velocity="1000000" />
+    </joint>
+    <joint name="arm_2_Revolute-10" type="revolute">
+        <origin xyz="0.038 0.0 0.00898067" rpy="3.141592653589793 -0.0 0.0" />
+        <parent link="arm_2" />
+        <child link="arm_3" />
+        <axis xyz="0.0 0.0 1.0" />
+        <limit lower="-1.570796" upper="1.570796" effort="1000000" velocity="1000000" />
+    </joint>
+    <joint name="base_Revolute-11" type="continuous">
+        <origin xyz="0.0 0.0 0.024" rpy="0.0 -0.0 0.0" />
+        <parent link="base" />
+        <child link="arm_1" />
+        <axis xyz="0.0 0.0 1.0" />
+    </joint>
 </robot>
