Commit message: Robot URDF with Fusion 360 Test complete!

File: install/urdf_test/share/urdf_test/urdf/my_robot.xacro (robot description, xacro)
@@ -136,10 +136,10 @@
     <link name="arm_3">
         <inertial>
-            <origin xyz="0.017021830705348132 2.2590601918467236e-18 0.003979455780812923" rpy="0.0 -0.0 0.0" />
-            <mass value="0.015207027813440301" />
-            <inertia ixx="1.1895476288949197e-07" iyy="1.9861577194252387e-06" izz="1.9861577267136794e-06" ixy="1.7430501486614956e-21" iyz="9.183549615799121e-41" ixz="-4.684356896112298e-17" />
+            <origin xyz="0.01847214368312333 5.422946197896389e-05 0.003970952850250537" rpy="0.0 -0.0 0.0" />
+            <mass value="0.016191593837877324" />
+            <inertia ixx="1.304180623419037e-07" iyy="2.5269144712693886e-06" izz="2.516463905029504e-06" ixy="-1.924174840835271e-08" iyz="1.1026562852339944e-10" ixz="2.993078018997173e-09" />
         </inertial>
         <visual name="arm_3_visual">
-            <origin xyz="-0.09049999658483847 2.259060191846725e-18 0.003979455781202988" rpy="1.232595164407831e-32 1.5707963267948966 0" />
+            <origin xyz="-0.09049999658483845 2.259060191846725e-18 0.003979455781202988" rpy="1.232595164407831e-32 1.5707963267948966 0" />
             <geometry>
                 <mesh filename="package://urdf_test/meshes/arm_3.stl" scale="0.001 0.001 0.001" />
@@ -147,7 +147,45 @@
         </visual>
         <collision name="arm_3_collision">
-            <origin xyz="-0.09049999658483847 2.259060191846725e-18 0.003979455781202988" rpy="1.232595164407831e-32 1.5707963267948966 0" />
+            <origin xyz="-0.09049999658483845 2.259060191846725e-18 0.003979455781202988" rpy="1.232595164407831e-32 1.5707963267948966 0" />
             <geometry>
                 <mesh filename="package://urdf_test/meshes/arm_3.stl" scale="0.001 0.001 0.001" />
+            </geometry>
+        </collision>
+    </link>
+    <link name="gripper_gear_1">
+        <inertial>
+            <origin xyz="0.0017362214484572204 -0.0002862433124168184 -0.002009304671236128" rpy="0.0 -0.0 0.0" />
+            <mass value="0.0006011056672916086" />
+            <inertia ixx="1.88772495882846e-09" iyy="8.211589146672423e-09" izz="9.349750078771848e-09" ixy="5.421138409108764e-10" iyz="1.6643901023854444e-10" ixz="-1.0055595168709039e-09" />
+        </inertial>
+        <visual name="gripper_gear_1_visual">
+            <origin xyz="0.0543908059196748 -0.12899144399999998 -0.003311543941894128" rpy="-1.5707963267948963 -0.0 0.0" />
+            <geometry>
+                <mesh filename="package://urdf_test/meshes/gripper_gear_1.stl" scale="0.001 0.001 0.001" />
+            </geometry>
+        </visual>
+        <collision name="gripper_gear_1_collision">
+            <origin xyz="0.0543908059196748 -0.12899144399999998 -0.003311543941894128" rpy="-1.5707963267948963 -0.0 0.0" />
+            <geometry>
+                <mesh filename="package://urdf_test/meshes/gripper_gear_1.stl" scale="0.001 0.001 0.001" />
+            </geometry>
+        </collision>
+    </link>
+    <link name="gripper_gear_2">
+        <inertial>
+            <origin xyz="-0.0017331970562074878 -0.0002862477685876463 -0.002009304708227388" rpy="0.0 -0.0 0.0" />
+            <mass value="0.0006011056445017347" />
+            <inertia ixx="1.88772494109159e-09" iyy="8.198613493250422e-09" izz="9.336774458920598e-09" ixy="-5.41043181725309e-10" iyz="1.6643898505927248e-10" ixz="1.0038072080775312e-09" />
+        </inertial>
+        <visual name="gripper_gear_2_visual">
+            <origin xyz="0.06143864417246264 -0.12899634400000004 -0.00331643944132532" rpy="-1.5707963267948963 -0.0 0.0" />
+            <geometry>
+                <mesh filename="package://urdf_test/meshes/gripper_gear_2.stl" scale="0.001 0.001 0.001" />
+            </geometry>
+        </visual>
+        <collision name="gripper_gear_2_collision">
+            <origin xyz="0.06143864417246264 -0.12899634400000004 -0.00331643944132532" rpy="-1.5707963267948963 -0.0 0.0" />
+            <geometry>
+                <mesh filename="package://urdf_test/meshes/gripper_gear_2.stl" scale="0.001 0.001 0.001" />
             </geometry>
         </collision>
@@ -198,3 +236,18 @@
         <axis xyz="0.0 0.0 1.0" />
     </joint>
+    <joint name="arm_3_Revolute-19" type="revolute">
+        <origin xyz="0.041335840000000006 -0.0032446199999999997 0.00039081000000000033" rpy="1.5707963267948966 1.5707963267948966 0" />
+        <parent link="arm_3" />
+        <child link="gripper_gear_1" />
+        <axis xyz="0.0 0.0 1.0" />
+        <limit lower="0.0" upper="1.710423" effort="1000000" velocity="1000000" />
+    </joint>
+    <joint name="arm_3_Revolute-20" type="revolute">
+        <origin xyz="0.04134074 -0.0032446199999999997 0.00742683" rpy="1.5707963267948966 1.5707963267948966 0" />
+        <parent link="arm_3" />
+        <child link="gripper_gear_2" />
+        <axis xyz="0.0 0.0 1.0" />
+        <limit lower="-1.710423" upper="0.0" effort="1000000" velocity="1000000" />
+        <mimic joint="arm_3_Revolute-19" multiplier="-1.0" offset="0.0" />
+    </joint>
 </robot>

Commit message: Working on new robot

File: install/urdf_test/share/urdf_test/urdf/my_robot.xacro (robot description, xacro)
@@ -1,4 +1,8 @@
 <?xml version='1.0' encoding='utf-8'?>
-<robot name="ros2_robot_test1">
+<robot name="my_robot">
+    <export>
+        <build_type>ament_cmake</build_type>
+        <gazebo_ros gazebo_model_path = "/home/user/Documents/ros2_ws/install/urdf_test/share/" />
+    </export>
     <link name="base">
         <inertial>
@@ -10,11 +14,14 @@
             <origin xyz="0.0 0.0 0.0" rpy="0.0 0.0 0.0" />
             <geometry>
-                <mesh filename="model://urdf_test/meshes/base.stl" scale="0.001 0.001 0.001" />
-            </geometry>
+                <mesh filename="file://$(find urdf_test)/meshes/base.stl" scale="0.001 0.001 0.001" />
+            </geometry>
+            <material name="Cyan">
+                <color rgba="0 1 1 1" />
+            </material>
         </visual>
         <collision name="base_collision">
             <origin xyz="0.0 0.0 0.0" rpy="0.0 0.0 0.0" />
             <geometry>
-                <mesh filename="model://urdf_test/meshes/base.stl" scale="0.001 0.001 0.001" />
+                <mesh filename="file://$(find urdf_test)/meshes/base.stl" scale="0.001 0.001 0.001" />
             </geometry>
         </collision>
@@ -29,11 +36,14 @@
             <origin xyz="0.05050000000000001 -1.6653345369377347e-18 0.005" rpy="3.141592653589793 -0.0 0.0" />
             <geometry>
-                <mesh filename="model://urdf_test/meshes/steering.stl" scale="0.001 0.001 0.001" />
-            </geometry>
+                <mesh filename="file://$(find urdf_test)/meshes/steering.stl" scale="0.001 0.001 0.001" />
+            </geometry>
+            <material name="Cyan">
+                <color rgba="0 1 1 1" />
+            </material>
         </visual>
         <collision name="steering_collision">
             <origin xyz="0.05050000000000001 -1.6653345369377347e-18 0.005" rpy="3.141592653589793 -0.0 0.0" />
             <geometry>
-                <mesh filename="model://urdf_test/meshes/steering.stl" scale="0.001 0.001 0.001" />
+                <mesh filename="file://$(find urdf_test)/meshes/steering.stl" scale="0.001 0.001 0.001" />
             </geometry>
         </collision>
@@ -48,11 +58,14 @@
             <origin xyz="-0.06302599985826682 -0.003489789468550507 0.0029999999999999983" rpy="-1.5707963267948966 -0.0 3.141592653589793" />
             <geometry>
-                <mesh filename="model://urdf_test/meshes/front_wheel.stl" scale="0.001 0.001 0.001" />
-            </geometry>
+                <mesh filename="file://$(find urdf_test)/meshes/front_wheel.stl" scale="0.001 0.001 0.001" />
+            </geometry>
+            <material name="Cyan">
+                <color rgba="0 1 1 1" />
+            </material>
         </visual>
         <collision name="front_wheel_collision">
             <origin xyz="-0.06302599985826682 -0.003489789468550507 0.0029999999999999983" rpy="-1.5707963267948966 -0.0 3.141592653589793" />
             <geometry>
-                <mesh filename="model://urdf_test/meshes/front_wheel.stl" scale="0.001 0.001 0.001" />
+                <mesh filename="file://$(find urdf_test)/meshes/front_wheel.stl" scale="0.001 0.001 0.001" />
             </geometry>
         </collision>
@@ -67,11 +80,14 @@
             <origin xyz="0.026000000372529027 -3.1840817234047667e-18 -0.02" rpy="1.5707963267948966 -0.0 3.141592653589793" />
             <geometry>
-                <mesh filename="model://urdf_test/meshes/right_wheel.stl" scale="0.001 0.001 0.001" />
-            </geometry>
+                <mesh filename="file://$(find urdf_test)/meshes/right_wheel.stl" scale="0.001 0.001 0.001" />
+            </geometry>
+            <material name="Cyan">
+                <color rgba="0 1 1 1" />
+            </material>
         </visual>
         <collision name="right_wheel_collision">
             <origin xyz="0.026000000372529027 -3.1840817234047667e-18 -0.02" rpy="1.5707963267948966 -0.0 3.141592653589793" />
             <geometry>
-                <mesh filename="model://urdf_test/meshes/right_wheel.stl" scale="0.001 0.001 0.001" />
+                <mesh filename="file://$(find urdf_test)/meshes/right_wheel.stl" scale="0.001 0.001 0.001" />
             </geometry>
         </collision>
@@ -86,11 +102,14 @@
             <origin xyz="-0.004341204506362234 0.02462019419217468 -0.02" rpy="-1.5707963267948966 -0.0 -1.396263401595464" />
             <geometry>
-                <mesh filename="model://urdf_test/meshes/left_wheel.stl" scale="0.001 0.001 0.001" />
-            </geometry>
+                <mesh filename="file://$(find urdf_test)/meshes/left_wheel.stl" scale="0.001 0.001 0.001" />
+            </geometry>
+            <material name="Cyan">
+                <color rgba="0 1 1 1" />
+            </material>
         </visual>
         <collision name="left_wheel_collision">
             <origin xyz="-0.004341204506362234 0.02462019419217468 -0.02" rpy="-1.5707963267948966 -0.0 -1.396263401595464" />
             <geometry>
-                <mesh filename="model://urdf_test/meshes/left_wheel.stl" scale="0.001 0.001 0.001" />
+                <mesh filename="file://$(find urdf_test)/meshes/left_wheel.stl" scale="0.001 0.001 0.001" />
             </geometry>
         </collision>
@@ -105,11 +124,14 @@
             <origin xyz="-1.1102230246251566e-18 0.0 -0.023" rpy="0.0 -0.0 0.0" />
             <geometry>
-                <mesh filename="model://urdf_test/meshes/arm_1.stl" scale="0.001 0.001 0.001" />
-            </geometry>
+                <mesh filename="file://$(find urdf_test)/meshes/arm_1.stl" scale="0.001 0.001 0.001" />
+            </geometry>
+            <material name="Cyan">
+                <color rgba="0 1 1 1" />
+            </material>
         </visual>
         <collision name="arm_1_collision">
             <origin xyz="-1.1102230246251566e-18 0.0 -0.023" rpy="0.0 -0.0 0.0" />
             <geometry>
-                <mesh filename="model://urdf_test/meshes/arm_1.stl" scale="0.001 0.001 0.001" />
+                <mesh filename="file://$(find urdf_test)/meshes/arm_1.stl" scale="0.001 0.001 0.001" />
             </geometry>
         </collision>
@@ -124,11 +146,14 @@
             <origin xyz="-0.05149999658483846 3.7085770201170125e-18 0.004980669999999999" rpy="3.141592653589793 -1.5707963267948966 0" />
             <geometry>
-                <mesh filename="model://urdf_test/meshes/arm_2.stl" scale="0.001 0.001 0.001" />
-            </geometry>
+                <mesh filename="file://$(find urdf_test)/meshes/arm_2.stl" scale="0.001 0.001 0.001" />
+            </geometry>
+            <material name="Cyan">
+                <color rgba="0 1 1 1" />
+            </material>
         </visual>
         <collision name="arm_2_collision">
             <origin xyz="-0.05149999658483846 3.7085770201170125e-18 0.004980669999999999" rpy="3.141592653589793 -1.5707963267948966 0" />
             <geometry>
-                <mesh filename="model://urdf_test/meshes/arm_2.stl" scale="0.001 0.001 0.001" />
+                <mesh filename="file://$(find urdf_test)/meshes/arm_2.stl" scale="0.001 0.001 0.001" />
             </geometry>
         </collision>
@@ -143,11 +168,14 @@
             <origin xyz="-0.09049999658483845 2.259060191846725e-18 0.003979455781202988" rpy="1.232595164407831e-32 1.5707963267948966 0" />
             <geometry>
-                <mesh filename="model://urdf_test/meshes/arm_3.stl" scale="0.001 0.001 0.001" />
-            </geometry>
+                <mesh filename="file://$(find urdf_test)/meshes/arm_3.stl" scale="0.001 0.001 0.001" />
+            </geometry>
+            <material name="Cyan">
+                <color rgba="0 1 1 1" />
+            </material>
         </visual>
         <collision name="arm_3_collision">
             <origin xyz="-0.09049999658483845 2.259060191846725e-18 0.003979455781202988" rpy="1.232595164407831e-32 1.5707963267948966 0" />
             <geometry>
-                <mesh filename="model://urdf_test/meshes/arm_3.stl" scale="0.001 0.001 0.001" />
+                <mesh filename="file://$(find urdf_test)/meshes/arm_3.stl" scale="0.001 0.001 0.001" />
             </geometry>
         </collision>
@@ -162,11 +190,14 @@
             <origin xyz="0.0543908059196748 -0.12899144399999998 -0.003311543941894128" rpy="-1.5707963267948963 -0.0 0.0" />
             <geometry>
-                <mesh filename="model://urdf_test/meshes/gripper_gear_1.stl" scale="0.001 0.001 0.001" />
-            </geometry>
+                <mesh filename="file://$(find urdf_test)/meshes/gripper_gear_1.stl" scale="0.001 0.001 0.001" />
+            </geometry>
+            <material name="Cyan">
+                <color rgba="0 1 1 1" />
+            </material>
         </visual>
         <collision name="gripper_gear_1_collision">
             <origin xyz="0.0543908059196748 -0.12899144399999998 -0.003311543941894128" rpy="-1.5707963267948963 -0.0 0.0" />
             <geometry>
-                <mesh filename="model://urdf_test/meshes/gripper_gear_1.stl" scale="0.001 0.001 0.001" />
+                <mesh filename="file://$(find urdf_test)/meshes/gripper_gear_1.stl" scale="0.001 0.001 0.001" />
             </geometry>
         </collision>
@@ -181,11 +212,14 @@
             <origin xyz="0.06143864417246264 -0.12899634400000004 -0.00331643944132532" rpy="-1.5707963267948963 -0.0 0.0" />
             <geometry>
-                <mesh filename="model://urdf_test/meshes/gripper_gear_2.stl" scale="0.001 0.001 0.001" />
-            </geometry>
+                <mesh filename="file://$(find urdf_test)/meshes/gripper_gear_2.stl" scale="0.001 0.001 0.001" />
+            </geometry>
+            <material name="Cyan">
+                <color rgba="0 1 1 1" />
+            </material>
         </visual>
         <collision name="gripper_gear_2_collision">
             <origin xyz="0.06143864417246264 -0.12899634400000004 -0.00331643944132532" rpy="-1.5707963267948963 -0.0 0.0" />
             <geometry>
-                <mesh filename="model://urdf_test/meshes/gripper_gear_2.stl" scale="0.001 0.001 0.001" />
+                <mesh filename="file://$(find urdf_test)/meshes/gripper_gear_2.stl" scale="0.001 0.001 0.001" />
             </geometry>
         </collision>
@@ -222,4 +256,5 @@
         <axis xyz="0.0 0.0 1.0" />
         <limit lower="-1.570796" upper="1.570796" effort="1000000" velocity="1000000" />
+        <dynamics damping="0.01" friction="0.01" />
     </joint>
     <joint name="arm_2_Revolute-10" type="revolute">
@@ -229,4 +264,5 @@
         <axis xyz="0.0 0.0 1.0" />
         <limit lower="-1.570796" upper="1.570796" effort="1000000" velocity="1000000" />
+        <dynamics damping="0.01" friction="0.01" />
     </joint>
     <joint name="base_Revolute-11" type="continuous">
@@ -235,4 +271,5 @@
         <child link="arm_1" />
         <axis xyz="0.0 0.0 1.0" />
+        <dynamics damping="0.01" friction="0.01" />
     </joint>
     <joint name="arm_3_Revolute-19" type="revolute">
@@ -242,4 +279,5 @@
         <axis xyz="0.0 0.0 1.0" />
         <limit lower="0.0" upper="1.710423" effort="1000000" velocity="1000000" />
+        <dynamics damping="0.01" friction="0.01" />
     </joint>
     <joint name="arm_3_Revolute-20" type="revolute">
@@ -250,4 +288,46 @@
         <limit lower="-1.710423" upper="0.0" effort="1000000" velocity="1000000" />
         <mimic joint="arm_3_Revolute-19" multiplier="-1.0" offset="0.0" />
-    </joint>
+        <dynamics damping="0.01" friction="0.01" />
+    </joint>
+    <gazebo>
+        <plugin name="gz::sim::systems::JointPositionController" filename="gz-sim-joint-position-controller-system">
+            <joint_name>arm_1_Revolute-9</joint_name>
+            <p_gain>5.0</p_gain>
+        </plugin>
+    </gazebo>
+    <gazebo>
+        <plugin name="gz::sim::systems::JointPositionController" filename="gz-sim-joint-position-controller-system">
+            <joint_name>arm_2_Revolute-10</joint_name>
+            <p_gain>5.0</p_gain>
+        </plugin>
+    </gazebo>
+    <gazebo>
+        <plugin name="gz::sim::systems::JointPositionController" filename="gz-sim-joint-position-controller-system">
+            <joint_name>base_Revolute-11</joint_name>
+            <p_gain>5.0</p_gain>
+        </plugin>
+    </gazebo>
+    <gazebo>
+        <plugin name="gz::sim::systems::DiffDrive" filename="gz-sim-diff-drive-system">
+            <left_joint>base_Revolute-3</left_joint>
+            <right_joint>base_Revolute-4</right_joint>
+            <wheel_separation>0.34</wheel_separation>
+            <wheel_radius>0.1</wheel_radius>
+            <frame_id>odom</frame_id>
+            <child_frame_id>base</child_frame_id>
+        </plugin>
+    </gazebo>
+    <gazebo>
+        <plugin name = "gz::sim::systems::JointStatePublisher" filename="gz-sim-joint-state-publisher-system">
+            <joint_name>base_Revolute-1</joint_name>
+            <joint_name>base_Revolute-3</joint_name>
+            <joint_name>base_Revolute-4</joint_name>
+            <joint_name>steering_Revolute-6</joint_name>
+            <joint_name>arm_1_Revolute-9</joint_name>
+            <joint_name>arm_2_Revolute-10</joint_name>
+            <joint_name>base_Revolute-11</joint_name>
+            <joint_name>arm_3_Revolute-19</joint_name>
+            <joint_name>arm_3_Revolute-20</joint_name>
+        </plugin>
+    </gazebo>
 </robot>
